Commit message: Add talos ati and imu

File: urdf/ft_sensors/ati.urdf.xacro (robot description, xacro)
@@ -31,5 +31,5 @@
         <origin xyz="0 0 0" rpy="0 0 0" />
         <geometry>
-          <mesh filename="package://pal_sea_arm_description/meshes/sensors/ati/ati_ft_sensor.stl"/>
+          <mesh filename="$(find pal_urdf_utils)/meshes/ft_sensors/ati_ft_sensor.stl"/>
         </geometry>
         <material name="pal/DarkGrey"/>

File: urdf/ft_sensors/rokubi.urdf.xacro (robot description, xacro)
@@ -24,5 +24,5 @@
         <origin xyz="0.0 0.0 0.0" rpy="0.0 0.0 0.0"/>
         <geometry>
-          <mesh filename="package://pal_sea_arm_description/meshes/sensors/rokubi/rokubi_ft_sensor.stl"/>
+          <mesh filename="$(find pal_urdf_utils)/meshes/ft_sensors/rokubi_ft_sensor.stl"/>
         </geometry>
         <material name="pal/DarkGrey"/>
