Commit message: Fix meshes paths

File: urdf/laser/ydlidar_tg15_laser.urdf.xacro (robot description, xacro)
@@ -21,5 +21,5 @@
         <origin xyz="0 0 0" rpy="0 0 0" />
         <geometry>
-          <mesh filename="$(find pal_urdf_utils)/meshes/laser/ydlidar.dae"/>
+          <mesh filename="package://pal_urdf_utils/meshes/laser/ydlidar.dae"/>
         </geometry>
         <material name="DarkGrey"/>

File: urdf/laser/ydlidar_tg30_laser.urdf.xacro (robot description, xacro)
@@ -21,5 +21,5 @@
         <origin xyz="0 0 0" rpy="0 0 0" />
         <geometry>
-          <mesh filename="$(find pal_urdf_utils)/meshes/laser/ydlidar.dae"/>
+          <mesh filename="package://pal_urdf_utils/meshes/laser/ydlidar.dae"/>
         </geometry>
         <material name="DarkGrey"/>

Commit message: fix error not visualize laser model in rviz

File: urdf/laser/ydlidar_tg15_laser.urdf.xacro (robot description, xacro)
@@ -25,4 +25,10 @@
         <material name="DarkGrey"/>
       </visual>
+      <collision>
+        <origin xyz="0 0 0" rpy="0 0 0" />
+        <geometry>
+          <mesh filename="package://pal_urdf_utils/meshes/laser/ydlidar.dae"/>
+        </geometry>
+      </collision>
     </link>
     <joint name="${name}_joint" type="fixed">
