Commit message: update mesh

File: urdf/camera/realsense_t265.urdf.xacro (robot description, xacro)
@@ -44,5 +44,5 @@
       <origin xyz="0 0 0" rpy="0 0 0"/>
         <geometry>
-            <mesh filename="package://realsense2_description_deprecated/meshes/t265.stl" />
+            <mesh filename="package://pal_urdf_utils/meshes/camera/t265.stl" />
         </geometry>
         <material name="${name}_aluminum"/>
@@ -51,5 +51,5 @@
         <origin xyz="0 0 0" rpy="0 0 0"/>
         <geometry>
-          <mesh filename="package://realsense2_description_deprecated/meshes/t265.stl" />
+          <mesh filename="package://pal_urdf_utils/meshes/camera/t265.stl" />
         </geometry>
       </collision>
